Commit message: changes

File: description/ros2_control/diffbot.ros2_control.xacro (robot description, xacro)
@@ -7,5 +7,5 @@
         <param name="left_wheel_name">left_wheel_joint</param>
         <param name="right_wheel_name">right_wheel_joint</param>
-        <param name="loop_rate">30</param>
+        <param name="loop_rate">9</param>
         <param name="device">/dev/ttyACM0</param>
         <param name="baud_rate">57600</param>

File: description/urdf/diffbot_description.urdf.xacro (robot description, xacro)
@@ -4,11 +4,11 @@
   <!-- Constants for robot dimensions -->
   <xacro:property name="PI" value="3.1415926535897931"/>
-  <xacro:property name="base_mass" value="0.3" /> <!-- arbitrary value for base mass -->
-  <xacro:property name="base_width" value="0.1" />
-  <xacro:property name="base_length" value="0.1" />
-  <xacro:property name="base_height" value="0.05" />
-  <xacro:property name="wheel_mass" value="0.3" /> <!-- arbitrary value for wheel mass -->
-  <xacro:property name="wheel_len" value="0.020" />
-  <xacro:property name="wheel_radius" value="0.015" />
+  <xacro:property name="base_mass" value="0.6" /> <!-- arbitrary value for base mass -->
+  <xacro:property name="base_width" value="0.2" />
+  <xacro:property name="base_length" value="0.2" />
+  <xacro:property name="base_height" value="0.10" />
+  <xacro:property name="wheel_mass" value="0.6" /> <!-- arbitrary value for wheel mass -->
+  <xacro:property name="wheel_len" value="0.040" />
+  <xacro:property name="wheel_radius" value="0.035" />
   <xacro:property name="caster_wheel_mass" value="0.1" /> <!-- arbitrary value for caster wheel mass -->
   <xacro:property name="caster_wheel_radius" value="0.015" />

Commit message: changes

File: description/ros2_control/diffbot.ros2_control.xacro (robot description, xacro)
@@ -8,5 +8,5 @@
         <param name="right_wheel_name">right_wheel_joint</param>
         <param name="loop_rate">9</param>
-        <param name="device">/dev/ttyACM0</param>
+        <param name="device">/dev/serial/by-id/usb-Arduino__www.arduino.cc__0043_242303036373511180D1-if00</param>
         <param name="baud_rate">57600</param>
         <param name="timeout_ms">1000</param>

File: description/urdf/diffbot_description.urdf.xacro (robot description, xacro)
@@ -4,13 +4,13 @@
   <!-- Constants for robot dimensions -->
   <xacro:property name="PI" value="3.1415926535897931"/>
-  <xacro:property name="base_mass" value="0.6" /> <!-- arbitrary value for base mass -->
-  <xacro:property name="base_width" value="0.2" />
-  <xacro:property name="base_length" value="0.2" />
-  <xacro:property name="base_height" value="0.10" />
+  <xacro:property name="base_mass" value="0.8" /> <!-- arbitrary value for base mass -->
+  <xacro:property name="base_width" value="0.16" />
+  <xacro:property name="base_length" value="0.19" />
+  <xacro:property name="base_height" value="0.07" />
   <xacro:property name="wheel_mass" value="0.6" /> <!-- arbitrary value for wheel mass -->
   <xacro:property name="wheel_len" value="0.040" />
   <xacro:property name="wheel_radius" value="0.035" />
   <xacro:property name="caster_wheel_mass" value="0.1" /> <!-- arbitrary value for caster wheel mass -->
-  <xacro:property name="caster_wheel_radius" value="0.015" />
+  <xacro:property name="caster_wheel_radius" value="0.007" />
   <xacro:property name="z_offset" value="-${base_height/2}" /> <!-- Space btw top of beam and the each joint -->
   <!-- Base Link -->

Commit message: changes

File: description/ros2_control/diffbot.ros2_control.xacro (robot description, xacro)
@@ -7,5 +7,5 @@
         <param name="left_wheel_name">left_wheel_joint</param>
         <param name="right_wheel_name">right_wheel_joint</param>
-        <param name="loop_rate">9</param>
+        <param name="loop_rate">10</param>
         <param name="device">/dev/serial/by-id/usb-Arduino__www.arduino.cc__0043_242303036373511180D1-if00</param>
         <param name="baud_rate">57600</param>

File: description/urdf/diffbot_description.urdf.xacro (robot description, xacro)
@@ -5,9 +5,9 @@
   <xacro:property name="PI" value="3.1415926535897931"/>
   <xacro:property name="base_mass" value="0.8" /> <!-- arbitrary value for base mass -->
-  <xacro:property name="base_width" value="0.16" />
-  <xacro:property name="base_length" value="0.19" />
-  <xacro:property name="base_height" value="0.07" />
-  <xacro:property name="wheel_mass" value="0.6" /> <!-- arbitrary value for wheel mass -->
-  <xacro:property name="wheel_len" value="0.040" />
+  <xacro:property name="base_width" value="0.15" />
+  <xacro:property name="base_length" value="0.20" />
+  <xacro:property name="base_height" value="0.11" />
+  <xacro:property name="wheel_mass" value="0.06" /> <!-- arbitrary value for wheel mass -->
+  <xacro:property name="wheel_len" value="0.07" />
   <xacro:property name="wheel_radius" value="0.035" />
   <xacro:property name="caster_wheel_mass" value="0.1" /> <!-- arbitrary value for caster wheel mass -->
